File: Eagle Files/driver_board.sch (EAGLE design)
At the start: 70 parts, among them Q1 TIP32, Q2 TIP32, Q3 TIP32, Q4 TIP32, Q5 TIP32, Q6 TIP32, Q7 TIP32, Q8 TIP32, U1 STP16CPP05MTR, U10 STP16CPP05MTR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

Commit message: Driver Board - Production Release
final board layout - release for production
Parts:
- removed X1: (no value), con-wago-500:W237-102
- added PWR: (no value), con-wago-500:W237-102
- added R21, R23, R25, R27, R29: 1K, adafruit:R-US_R0805
- added R24, R26, R28: 2K, adafruit:R-US_R0805
- C1: value (none) -> 0.01; MF AVX CORPORATION -> (none); MPN 0805ZC105KAT2A -> MCCA001261; OC_NEWARK 22C5489 -> 23T7439
- C10, C11, C12, C13, C2, C3, C4, C5, C6, C7, C8, C9: MF AVX CORPORATION -> (none); MPN 0805ZC105KAT2A -> MCCA001261; OC_NEWARK 22C5489 -> 23T7439
- R1: value 1K -> 220; MPN MC01W080511K -> MCHP05W4F2200T5E; OC_NEWARK 07W5249 -> 01N7012
- R13: value 1k -> 1K; MPN (none) -> MC01W080511K; OC_NEWARK unknown -> 07W5249
- R14, R16, R18, R20: value 1k -> 2K
- R15, R17, R19: value 1k -> 1K
- R22: value 220 -> 2K; MPN MCHP05W4F2200T5E -> (none); OC_NEWARK 01N7012 -> unknown
Connections:
- net +3V3: now also PWR-1.KL, R1.2, R14.1, R16.1, R18.1, R20.1, R22.1, R24.1, R26.1, R28.1; no longer R22.2, X1-1.KL
- net CLK: now also SV13.2; no longer SV14.2
- net GND: now also PWR-2.KL, R13.1; no longer R1.1, X1-2.KL
- net LE: now also SV13.4; no longer SV14.4
- net N$108: now also R7.2; no longer R6.2
- net N$126: now also R8.2; no longer R7.2
- net N$144: now also R9.2; no longer R8.2
- net N$162: now also R10.2; no longer R9.2
- net N$180: now also R11.2; no longer R10.2
- net N$19: now also R2.2; no longer R1.2
- net N$198: now also R12.2; no longer R11.2
- net N$216: now also R13.2; no longer R12.2
- net N$226: now also SV14.1; no longer SV13.1
- net N$227: now also SV14.3; no longer SV13.3
- net N$228: now also SV14.5; no longer SV13.5
- net N$229: now also SV14.7; no longer SV13.7
- net N$230: now also SV14.9; no longer SV13.9
- net N$231: now also SV14.11; no longer SV13.11
- net N$232: now also R15.1; no longer R13.1
- net N$233: now also SV14.13; no longer SV13.13
- net N$234: now also SV14.15; no longer SV13.15
- net N$235: now also R29.1; no longer R20.1
- net N$236: now also R27.1; no longer R19.1
- net N$237: now also R25.1; no longer R18.1
- net N$238: now also R23.1; no longer R17.1
- net N$239: now also R21.1; no longer R16.1
- net N$240: now also R19.1; no longer R15.1
- net N$241: now also R17.1; no longer R14.1
- net N$243: now also R28.2, R29.2, SV13.15; no longer R20.2, SV14.15
- net N$244: now also R1.1; no longer R22.1
- net N$245: now also R26.2, R27.2, SV13.13; no longer R19.2, SV14.13
- net N$246: now also R24.2, R25.2, SV13.11; no longer R18.2, SV14.11
- net N$247: now also R22.2, R23.2, SV13.9; no longer R17.2, SV14.9
- net N$248: now also R20.2, R21.2, SV13.7; no longer R16.2, SV14.7
- net N$249: now also R18.2, R19.2, SV13.5; no longer R15.2, SV14.5
- net N$250: now also R16.2, R17.2, SV13.3; no longer R14.2, SV14.3
- net N$251: now also R14.2, R15.2, SV13.1; no longer R13.2, SV14.1
- net N$36: now also R3.2; no longer R2.2
- net N$54: now also R4.2; no longer R3.2
- net N$72: now also R5.2; no longer R4.2
- net N$90: now also R6.2; no longer R5.2
- net SDI_B: now also SV13.12; no longer SV14.12
- net SDI_G: now also SV13.10; no longer SV14.10
- net SDI_R: now also SV13.8; no longer SV14.8
- net ~OE: now also SV13.6; no longer SV14.6
Other:
- moved on the sheet: C1, C10, C11, C12, C13, C2, C3, C4, C5, C6, C7, C8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
